File: ESP32-S3-HUB75-Driver.kicad_pcb (KiCad board)
At the start: 2 copper layers, 62 x 100 mm, 93 parts, among them J1 Conn_02x08_Odd_Even, J2 Barrel_Jack_Switch, J4 USB_C_Receptacle_USB2.0, J5 USB_B_Mini, J6 Conn_01x04_Socket, Q1 DMP3036SSD, Q2 DMP3036SSD, SW1 SW_SPST, SW2 SW_SPST, SW3 SW_SPST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

Commit message: updated schematic to look neater
Connections:
- U1 pad 20: unconnected-(U1-IO12-Pad20) -> /ADDRC_3V
- U1 pad 24: /ADDRC_3V -> /CLK_3V
- U1 pad 38: /CLK_3V -> unconnected-(U1-IO2-Pad38)
- U3 pad 6: /ADDRC_3V -> /CLK_3V
Routing:
- net /CLK_3V: track 0.00 -> 19.7 mm
- net /ADDRC_3V: track 19.7 -> 0.00 mm
Changed lines of the file:
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@@
   (net 60 "unconnected-(U1-IO10-Pad18)")
   (net 61 "unconnected-(U1-IO11-Pad19)")
-  (net 62 "unconnected-(U1-IO12-Pad20)")
+  (net 62 "unconnected-(U1-IO2-Pad38)")
   (net 63 "Net-(U4-SS)")
   (net 64 "/ADDRE_3V")
@@
       (net 67 "/ADDRA_3V") (pinfunction "A3") (pintype "passive"))
     (pad "6" smd roundrect (at -2.8625 0.325 270) (size 1.475 0.4) (layers "F.Cu" "F.Paste" "F.Mask") (roundrect_rratio 0.25)
-      (net 66 "/ADDRC_3V") (pinfunction "A4") (pintype "passive"))
+      (net 79 "/CLK_3V") (pinfunction "A4") (pintype "passive"))
     (pad "7" smd roundrect (at -2.8625 0.975 270) (size 1.475 0.4) (layers "F.Cu" "F.Paste" "F.Mask") (roundrect_rratio 0.25)
       (net 65 "/LAT_3V") (pinfunction "A5") (pintype "passive"))
@@
       (net 61 "unconnected-(U1-IO11-Pad19)") (pinfunction "IO11") (pintype "bidirectional"))
     (pad "20" smd rect locked (at -0.635 12.5 270) (size 1.5 0.9) (layers "F.Cu" "F.Paste" "F.Mask")
-      (net 62 "unconnected-(U1-IO12-Pad20)") (pinfunction "IO12") (pintype "bidirectional"))
+      (net 66 "/ADDRC_3V") (pinfunction "IO12") (pintype "bidirectional"))
     (pad "21" smd rect locked (at 0.635 12.5 270) (size 1.5 0.9) (layers "F.Cu" "F.Paste" "F.Mask")
       (net 58 "/OE_3V") (pinfunction "IO13") (pintype "bidirectional"))
@@
       (net 65 "/LAT_3V") (pinfunction "IO21") (pintype "bidirectional"))
     (pad "24" smd rect locked (at 4.445 12.5 270) (size 1.5 0.9) (layers "F.Cu" "F.Paste" "F.Mask")
-      (net 66 "/ADDRC_3V") (pinfunction "IO47") (pintype "bidirectional"))
+      (net 79 "/CLK_3V") (pinfunction "IO47") (pintype "bidirectional"))
     (pad "25" smd rect locked (at 5.715 12.5 270) (size 1.5 0.9) (layers "F.Cu" "F.Paste" "F.Mask")
       (net 67 "/ADDRA_3V") (pinfunction "IO48") (pintype "bidirectional"))
@@
       (net 100 "/ESP_TXD") (pinfunction "TXD0") (pintype "bidirectional"))
     (pad "38" smd rect locked (at 8.75 -2.72) (size 1.5 0.9) (layers "F.Cu" "F.Paste" "F.Mask")
-      (net 79 "/CLK_3V") (pinfunction "IO2") (pintype "bidirectional"))
+      (net 62 "unconnected-(U1-IO2-Pad38)") (pinfunction "IO2") (pintype "bidirectional"))
     (pad "39" smd rect locked (at 8.75 -3.99) (size 1.5 0.9) (layers "F.Cu" "F.Paste" "F.Mask")
       (net 80 "/IO1") (pinfunction "IO1") (pintype "bidirectional"))
@@
       (net 41 "/Power and USB Inputs/VSENSE_USBPD") (pinfunction "PA3") (pintype "unspecified"))
     (pad "9" smd roundrect (at -0.8 1.9375 90) (size 0.2 0.825) (layers "F.Cu" "F.Paste" "F.Mask") (roundrect_rratio 0.25)
-      (net 85 "/Power and USB Inputs/CS") (pinfunction "PA4") (pintype "unspecified"))
+      (net 85 "/Power and USB Inputs/CS") (pinfunction "PA4") (pintype "unspecified+no_connect"))
     (pad "10" smd roundrect (at -0.4 1.9375 90) (size 0.2 0.825) (layers "F.Cu" "F.Paste" "F.Mask") (roundrect_rratio 0.25)
-      (net 86 "/Power and USB Inputs/SCK") (pinfunction "PA5") (pintype "unspecified"))
+      (net 86 "/Power and USB Inputs/SCK") (pinfunction "PA5") (pintype "unspecified+no_connect"))
     (pad "11" smd roundrect (at 0 1.9375 90) (size 0.2 0.825) (layers "F.Cu" "F.Paste" "F.Mask") (roundrect_rratio 0.25)
-      (net 87 "/Power and USB Inputs/MISO") (pinfunction "PA6") (pintype "unspecified"))
+      (net 87 "/Power and USB Inputs/MISO") (pinfunction "PA6") (pintype "unspecified+no_connect"))
     (pad "12" smd roundrect (at 0.4 1.9375 90) (size 0.2 0.825) (layers "F.Cu" "F.Paste" "F.Mask") (roundrect_rratio 0.25)
-      (net 88 "/Power and USB Inputs/MOSI") (pinfunction "PA7") (pintype "unspecified"))
+      (net 88 "/Power and USB Inputs/MOSI") (pinfunction "PA7") (pintype "unspecified+no_connect"))
     (pad "13" smd roundrect (at 0.8 1.9375 90) (size 0.2 0.825) (layers "F.Cu" "F.Paste" "F.Mask") (roundrect_rratio 0.25)
       (net 89 "unconnected-(U7-PB0-Pad13)") (pinfunction "PB0") (pintype "unspecified+no_connect"))
@@
   (segment (start 106.425 90.5375) (end 106.425 89.125) (width 0.2032) (layer "F.Cu") (net 65))
   (segment (start 96.975 79.675) (end 96.975 74.5) (width 0.2032) (layer "F.Cu") (net 65))
-  (segment (start 98.245 80.045) (end 98.245 74.5) (width 0.2032) (layer "F.Cu") (net 66))
-  (segment (start 107.075 88.875) (end 98.245 80.045) (width 0.2032) (layer "F.Cu") (net 66))
-  (segment (start 107.075 90.5375) (end 107.075 88.875) (width 0.2032) (layer "F.Cu") (net 66))
   (segment (start 99.515 80.515) (end 99.515 74.5) (width 0.2032) (layer "F.Cu") (net 67))
   (segment (start 107.725 88.725) (end 99.515 80.515) (width 0.2032) (layer "F.Cu") (net 67))
@@
   (via (at 104.5 59.5) (size 0.6) (drill 0.3) (layers "F.Cu" "B.Cu") (net 78))
   (segment (start 100.5 59.5) (end 104.5 59.5) (width 0.25) (layer "B.Cu") (net 78))
+  (segment (start 98.245 80.045) (end 98.245 74.5) (width 0.2032) (layer "F.Cu") (net 79))
+  (segment (start 107.075 88.875) (end 98.245 80.045) (width 0.2032) (layer "F.Cu") (net 79))
+  (segment (start 107.075 90.5375) (end 107.075 88.875) (width 0.2032) (layer "F.Cu") (net 79))
   (segment (start 106.2 59.275) (end 104.935 58.01) (width 0.25) (layer "F.Cu") (net 80))
   (segment (start 104.935 58.01) (end 102.55 58.01) (width 0.25) (layer "F.Cu") (net 80))
