File: TPS51385.kicad_sch (KiCad schematic)
At the start: 15 parts, among them U4 TPS51385RJNR

Commit message: updated schematic to look neater
Parts:
- C10: value 0402,100nF,50V,X7R -> 0603,100nF,50V,X7R
- C15: value 0402,100nF,16V,X7R -> 0603,100nF,50V,X7R
- C16: value 0402,22pF,50V,C0G -> 0603,22pF,50V,C0G
- C9: value 0402,1uF,25V,X5R -> 0603,1uF,50V,X5R
- R17: value 0402,49.9k -> 0603,49.9k
- R18: value 0402,6.8k -> 0603,6.8k
Other:
- note added: "CHANGELOG/NOTES REV A01: Initial Design"
Changed lines of the file:
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@@
   (paper "USLetter")
   (title_block
-    (date "2024-01-28")
+    (date "2024-02-03")
     (rev "A01")
   )
@@
   (wire (pts (xy 203.2 100.33) (xy 203.2 107.95))
     (stroke (width 0) (type default))
+  )
+  (text "CHANGELOG/NOTES\n\nREV A01: Initial Design\n" (at 16.51 25.4 0)
+    (effects (font (size 1.27 1.27)) (justify left bottom))
   )
   (hierarchical_label "VIN" (shape input) (at 59.69 93.98 180) (fields_autoplaced)
@@
       (effects (font (size 0.8 0.8)) (justify left))
     )
-    (property "Value" "0402,100nF,50V,X7R " (at 135.89 96.52 0)
+    (property "Value" "0603,100nF,50V,X7R " (at 135.89 96.52 0)
       (effects (font (size 0.8 0.8)) (justify left))
     )
@@
       (effects (font (size 0.8 0.8)) (justify left))
     )
-    (property "Value" "0402,22pF,50V,C0G " (at 135.89 106.68 0)
+    (property "Value" "0603,22pF,50V,C0G " (at 135.89 106.68 0)
       (effects (font (size 0.8 0.8)) (justify left))
     )
@@
       (effects (font (size 0.8 0.8)) (justify left))
     )
-    (property "Value" "0402,1uF,25V,X5R " (at 77.47 115.57 0)
+    (property "Value" "0603,1uF,50V,X5R " (at 77.47 115.57 0)
       (effects (font (size 0.8 0.8)) (justify left))
     )
@@
       (effects (font (size 0.8 0.8)) (justify left))
     )
-    (property "Value" "0402,49.9k" (at 157.48 105.41 0)
+    (property "Value" "0603,49.9k" (at 157.48 105.41 0)
       (effects (font (size 0.8 0.8)) (justify left))
     )
@@
       (effects (font (size 0.8 0.8)) (justify left))
     )
-    (property "Value" "0402,100nF,16V,X7R " (at 134.62 119.38 0)
+    (property "Value" "0603,100nF,50V,X7R " (at 134.62 119.38 0)
       (effects (font (size 0.8 0.8)) (justify left))
     )
@@
       (effects (font (size 0.8 0.8)) (justify left))
     )
-    (property "Value" "0402,6.8k" (at 157.48 118.11 0)
-      (effects (font (size 0.8 0.8)) (justify left))
-    )
+    (property "Value" "0603,6.8k" (at 157.48 118.11 0)
+      (effects (font (size 0.8 0.8)) (justify left))
+    )
