File: Rev B/PowerMux.kicad_sch (KiCad schematic)
At the start: 50 parts, among them J1 USB4105, J2 Conn_02x05_Odd_Even, J9 Barrel_Jack, Q3 DMP3036SSD, SW1 PTS810 SJM, U11 L78L05_SOT89, U4 CH32X035G8U6, U8 AO3400A, U9 AO3400A

Commit message: B02: edited passive values
HSS slew rate edited by replacing slew-rate limiting capacitor to 4.7uF/35V
24V LED resistor changed to 10K to not burn an LED
Resistor divider for voltage sense edited to 18K/3,3K
Parts:
- C3, C8: value 0603,100nF,50V,X7R -> 0603,4.7uF,35V,X5R; LCSC C14663 -> (none); MFG YAGEO -> Samsung Electro-Mechanics; MFGPN CC0603KRX7R9BB104 -> CL10A475KL8NRNC
- R1, R12: value 0603,10k -> 0603,18k; LCSC C25804 -> C25810; MFGPN 0603WAF1002T5E -> 0603WAF1802T5E
- R11, R13: value 0603,1k -> 0603,3.3k; LCSC C21190 -> C22978; MFGPN 0603WAF1001T5E -> 0603WAF3301T5E
- R21, R22, R23: value 0603,1k -> 0603,10k; LCSC C21190 -> C25804; MFGPN 0603WAF1001T5E -> 0603WAF1002T5E
Other:
- note added: "Capacitance edited to modify slew rate"
- note added: "Divider ratio changed in B02"
- note added: "Resistor bumped to 10K for less bright LED"
